File: Benchtop ECEA PCB.kicad_sch (KiCad schematic)
At the start: 0 parts

Commit message: Added basic components for some workshop functionality
Parts:
- added J1: Conn_02x04_Odd_Even, symbol Connector_Generic:Conn_02x04_Odd_Even
- added TP1, TP2: TestPoint, symbol Connector:TestPoint
- added U1: 74LS48, symbol 74xx:74LS48
- added U2: HDSP-A151, Display_7Segment:HDSP-A151, symbol Display_Character:HDSP-A151
- added U3: LT1962-5, Package_SO:MSOP-8_3x3mm_P0.65mm, symbol Regulator_Linear:LT1962-5
Connections:
- new net +5V: TP1.1
- new net GND: TP2.1
Other:
- note added: "555 Timer"
- note added: "7-Segment"
- note added: "Power connector / LDO (5v)"

Commit message: Added pot
Parts:
- added R1: 10k, symbol Device:R_US
- added RV1: 10k, symbol Device:R_Potentiometer_US
- added TP3: +5v, symbol Connector:TestPoint
- added TP4: Vpot, symbol Connector:TestPoint
- added TP5: GND, symbol Connector:TestPoint
- TP1: value TestPoint -> +5v
- TP2: value TestPoint -> GND
Connections:
- net +5V: now also R1.1, TP3.1
- net GND: now also RV1.2, TP5.1
- new net: R1.2, RV1.1, TP4.1
- no-connect marks 0 -> 1
Other:
- note added: "Potentiometer voltage divider"
- note added: "Trough-hole testpoints for power connector"

Commit message: LDO Finished
Parts:
- added C1: 1uF, symbol Device:C
- added C2: 100nF, symbol Device:C
- added C3: 10uF, symbol Device:C_Polarized_US
Connections:
- net +5V: now also U3.1 (OUT), C3.1; no longer TP1.1
- net GND: now also U3.4 (GND), C1.2, C3.2
- net at U3.2 (SENSE): now also C2.1
- net at U3.3 (BYP): now also C2.2
- net VCC: now reaches U3.5 (~{SHDN})
- net VCC: now also TP1.1, U3.8 (IN), C1.1
